File: _autosave-Kicad-EffectsUnit1.kicad_pcb (KiCad board)
At the start: 2 copper layers, 100 x 100 mm, 171 parts, among them J101 In7, J102 Doepfer connector, J103 Vin 7-12v, J104 In6, J105 In3, J106 Out10, J107 Out11, J108 Out9, J109 Out6, J110 Power Conn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

Commit message: sch pinout
Parts:
- removed SW103: Dist 10, AJ-Dropbox-Kicad:SPDTx2
- SW101: value Dist 6 -> Dist 10
Connections:
- SW101 pad 4: (no net) -> Net-(R117-Pad2)
- SW101 pad 5: (no net) -> Net-(D110-Pad1)
- SW101 pad 6: (no net) -> GND
Changed lines of the file:
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@@
     (tracks 0)
     (zones 0)
-    (modules 171)
+    (modules 170)
     (nets 104)
   )
@@
       (effects (font (size 1 1) (thickness 0.15)))
     )
-    (fp_text value "Dist 6" (at 0 -8) (layer F.SilkS)
+    (fp_text value "Dist 10" (at 0 -8) (layer F.SilkS)
       (effects (font (size 1 1) (thickness 0.15)))
     )
@@
     (fp_circle (center 0 0) (end 0.5 0) (layer F.Fab) (width 0.2))
     (fp_circle (center 0 0) (end 3 0) (layer F.Fab) (width 0.2))
-    (pad 5 thru_hole oval (at 2.794 0) (size 3.9 2.5) (drill oval 2.55 1.15) (layers *.Cu *.Mask))
-    (pad 4 thru_hole oval (at 2.794 3.81) (size 3.9 2.5) (drill oval 2.55 1.15) (layers *.Cu *.Mask))
-    (pad 6 thru_hole oval (at 2.794 -3.938) (size 3.9 2.5) (drill oval 2.55 1.15) (layers *.Cu *.Mask))
+    (pad 5 thru_hole oval (at 2.794 0) (size 3.9 2.5) (drill oval 2.55 1.15) (layers *.Cu *.Mask)
+      (net 36 "Net-(D110-Pad1)"))
+    (pad 4 thru_hole oval (at 2.794 3.81) (size 3.9 2.5) (drill oval 2.55 1.15) (layers *.Cu *.Mask)
+      (net 50 "Net-(R117-Pad2)"))
+    (pad 6 thru_hole oval (at 2.794 -3.938) (size 3.9 2.5) (drill oval 2.55 1.15) (layers *.Cu *.Mask)
+      (net 2 GND))
     (pad 1 thru_hole oval (at -2.794 3.81) (size 3.9 2.5) (drill oval 2.55 1.15) (layers *.Cu *.Mask)
       (net 49 "Net-(R115-Pad2)"))
@@
     )
   )
-  (module AJ-Dropbox-Kicad:SPDTx2 (layer F.Cu)
-    (at 151.550001 170.958001)
-    (fp_text reference SW103 (at 0 2.413) (layer F.SilkS)
-      (effects (font (size 1 1) (thickness 0.15)))
-    )
-    (fp_text value "Dist 10" (at 0 -2.286) (layer F.Fab)
-      (effects (font (size 1 1) (thickness 0.15)))
-    )
-    (fp_circle (center 0 0) (end 3 0) (layer F.Fab) (width 0.2))
-    (fp_circle (center 0 0) (end 0.5 0) (layer F.Fab) (width 0.2))
-    (fp_line (start 0 0.5) (end 0 -0.5) (layer F.Fab) (width 0.2))
-    (fp_line (start 3.95 -6.6) (end -3.95 -6.6) (layer F.Fab) (width 0.2))
-    (fp_line (start -3.95 6.6) (end 3.95 6.6) (layer F.Fab) (width 0.2))
-    (fp_line (start 3.95 6.6) (end 3.95 -6.6) (layer F.Fab) (width 0.2))
-    (fp_line (start -3.95 -6.6) (end -3.95 6.6) (layer F.Fab) (width 0.2))
-    (fp_line (start -0.5 0) (end 0.5 0) (layer F.Fab) (width 0.2))
-    (fp_line (start -5.588 6.858) (end 5.588 6.858) (layer F.SilkS) (width 0.2))
-    (fp_line (start -5.588 -6.842) (end -5.588 6.858) (layer F.SilkS) (width 0.2))
-    (fp_line (start 5.588 6.842) (end 5.588 -6.858) (layer F.SilkS) (width 0.2))
-    (fp_line (start 5.588 -6.858) (end -5.588 -6.858) (layer F.SilkS) (width 0.2))
-    (fp_line (start -6 6.85) (end 6 6.85) (layer F.CrtYd) (width 0.2))
-    (fp_line (start -6 -6.85) (end -6 6.85) (layer F.CrtYd) (width 0.2))
-    (fp_line (start 0 0.5) (end 0 -0.5) (layer F.CrtYd) (width 0.2))
-    (fp_line (start 6 -6.85) (end -6 -6.85) (layer F.CrtYd) (width 0.2))
-    (fp_line (start 6 6.85) (end 6 -6.85) (layer F.CrtYd) (width 0.2))
-    (fp_line (start -0.5 0) (end 0.5 0) (layer F.CrtYd) (width 0.2))
-    (pad 2 thru_hole oval (at -2.794 0) (size 3.9 2.5) (drill oval 2.55 1.15) (layers *.Cu *.Mask)
-      (net 36 "Net-(D110-Pad1)"))
-    (pad 3 thru_hole oval (at -2.794 -3.938) (size 3.9 2.5) (drill oval 2.55 1.15) (layers *.Cu *.Mask)
-      (net 2 GND))
-    (pad 1 thru_hole oval (at -2.794 3.81) (size 3.9 2.5) (drill oval 2.55 1.15) (layers *.Cu *.Mask)
-      (net 50 "Net-(R117-Pad2)"))
-    (pad 6 thru_hole oval (at 2.794 -3.938) (size 3.9 2.5) (drill oval 2.55 1.15) (layers *.Cu *.Mask))
-    (pad 4 thru_hole oval (at 2.794 3.81) (size 3.9 2.5) (drill oval 2.55 1.15) (layers *.Cu *.Mask))
-    (pad 5 thru_hole oval (at 2.794 0) (size 3.9 2.5) (drill oval 2.55 1.15) (layers *.Cu *.Mask))
-    (model ${KIPRJMOD}/Local.pretty/SPDT.step
-      (at (xyz 0 0 0))
-      (scale (xyz 1 1 1))
-      (rotate (xyz 0 0 0))
-    )
-  )
   (module Rotary_Encoder:RotaryEncoder_Alps_EC11E-Switch_Vertical_H20mm (layer F.Cu)
     (at 100.525001 168.625001)
@@
       (effects (font (size 1 1) (thickness 0.15)))
     )
-    (fp_text value "Dist 10" (at 0 -2.286) (layer F.Fab)
+    (fp_text value "Dist 10" (at 0 -2.286) (layer F.SilkS)
       (effects (font (size 1 1) (thickness 0.15)))
     )
