File: _autosave-Kicad-EffectsUnit1.kicad_pcb (KiCad board)
At the start: 2 copper layers, 100 x 100 mm, 161 parts, among them J101 In7, J102 Doepfer connector, J104 In6, J105 In3, J106 Out10, J107 Out11, J108 Out9, J109 Out6, J201 In, J202 Out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

Commit message: GNDS and GNDA
Parts:
- removed U201: TL072, AJ-Dropbox-Kicad:AJ_SO-8_5.3x6.2mm_P1.27mm
- U202: moved to F.Cu
- moved C210 44.2 mm to (156.0, 55.0), turned to 90 degrees
- moved C201 35.3 mm to (144.0, 53.0), turned to 270 degrees
- moved U202 18.0 mm to (146.0, 94.0)

Commit message: misc
Parts:
- removed C203, C204, C207, C208, C209: 100n, Capacitor_SMD:C_0805_2012Metric_Pad1.15x1.40mm_HandSolder
- removed C206: 100uF 16v, Capacitor_THT:CP_Radial_D5.0mm_P2.50mm
- removed D203: 1N1007, Diode_SMD:D_SOD-123
- added C301: 100uF 16v, Capacitor_THT:CP_Radial_D5.0mm_P2.50mm, F.Cu at (228.7, 60.8)
- added C302: 100n, Capacitor_SMD:C_0805_2012Metric_Pad1.15x1.40mm_HandSolder, F.Cu at (209.9, 72.8)
- added C303: 100n, Capacitor_SMD:C_0805_2012Metric_Pad1.15x1.40mm_HandSolder, F.Cu at (221.7, 72.5)
- added C304: 100n, Capacitor_SMD:C_0805_2012Metric_Pad1.15x1.40mm_HandSolder, F.Cu at (232.8, 64.5)
- added C305: 100uF 16v, Capacitor_THT:CP_Radial_D5.0mm_P2.50mm, F.Cu at (221.4, 64.0)
- added C306: 100uF 16v, Capacitor_THT:CP_Radial_D5.0mm_P2.50mm, F.Cu at (215.8, 69.6)
- added C307: 100n, Capacitor_SMD:C_0805_2012Metric_Pad1.15x1.40mm_HandSolder, F.Cu at (226.5, 71.7)
- added C308: 100n, Capacitor_SMD:C_0805_2012Metric_Pad1.15x1.40mm_HandSolder, F.Cu at (231.2, 69.3)
- added C309: 100n, Capacitor_SMD:C_0805_2012Metric_Pad1.15x1.40mm_HandSolder, F.Cu at (232.8, 66.5)
- added C310: 100uF 16v, Capacitor_THT:CP_Radial_D5.0mm_P2.50mm, F.Cu at (215.8, 64.0)
- added D301: 1N1007, Diode_SMD:D_SOD-123, F.Cu at (227.0, 69.5)
- added D302: 1N1007, Diode_SMD:D_SOD-123, F.Cu at (222.2, 70.3)
- added D303: 1N1007, Diode_SMD:D_SOD-123, F.Cu at (222.2, 68.0)
- added D304: 5v6, Diode_SMD:D_MiniMELF_Handsoldering, F.Cu at (220.6, 59.6)
- added P301: HEADER_2x5_Doepfer, Connector_PinHeader_2.54mm:PinHeader_2x05_P2.54mm_Vertical, F.Cu at (209.8, 59.8)
- added Q301: BC337, Package_TO_SOT_THT:TO-92_Inline, F.Cu at (226.9, 66.3)
- added R301: 10k, Resistor_SMD:R_0805_2012Metric_Pad1.15x1.40mm_HandSolder, F.Cu at (230.2, 71.7)
- added R302: 0R, Resistor_SMD:R_0805_2012Metric_Pad1.15x1.40mm_HandSolder, F.Cu at (234.0, 71.3)
- D204: footprint Diode_SMD:D_MELF-RM10_Universal_Handsoldering -> Diode_SMD:D_MiniMELF_Handsoldering
- Q201: moved to F.Cu
- RV202: footprint Potentiometer_THT:Potentiometer_China_RK09_Single_Vertical_AJ -> Potentiometer_THT:Potentiometer_Alps_RK09K_Single_Vertical
- moved C212 127.3 mm to (152.0, 145.0)
- moved R203 125.8 mm to (152.0, 142.8)
- moved C225 94.1 mm to (148.0, 112.8), turned to 90 degrees
- moved C224 89.8 mm to (151.5, 110.5), turned to 90 degrees
- moved R207 86.2 mm to (163.2, 97.0)
- moved R206 86.0 mm to (167.2, 99.5)
- moved C220 85.2 mm to (156.5, 106.8)
- moved R205 84.5 mm to (163.2, 94.8)
- moved C202 84.3 mm to (148.0, 97.5), turned to 90 degrees
- moved R212 83.8 mm to (156.5, 104.2), turned to 180 degrees
- moved C211 83.3 mm to (163.1, 102.4)
- moved R208 81.5 mm to (167.2, 97.0), turned to 180 degrees
- moved C215 77.7 mm to (144.0, 96.5), turned to 270 degrees
- moved R214 75.7 mm to (145.5, 82.5)
- moved C222 75.1 mm to (164.0, 87.2)
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Connections:
- net -12Vb renamed Net-(P201-Pad1)
- C202 pad 2: +12Vb -> +5VA
- C222 pad 2: GND -> GNDA
- RV202 pad 3: GND -> GNDA
