File: _autosave-Kicad-EffectsUnit1.kicad_pcb (KiCad board)
At the start: 2 copper layers, 100 x 100 mm, 216 parts, among them J101 In7, J102 Doepfer connector, J104 In6, J105 In3, J106 Out10, J107 Out11, J108 Out9, J109 Out6, J201 In, J202 Out, J203 Conn_01x02_Male, J301 ClockOut, J302 Doepfer connector, J303 ClockIn, J304 Out0, J305 Out1, J306 Out2, J307 Out3, J308 Out4, J309 Out5, J310 Out6, J311 Out7, J312 Out8, J313 Out9, J314 Reset, P201 HEADER_2x5_Doepfer, P301 HEADER_2x5_Doepfer, Q201 BC337, Q202 PZT2222A, Q203 PZT2222A, Q301 BC337, SW101 Dist 6, SW102 Crush A6, SW104 Rotary_Encoder_Switch, SW105 Dist 10, SW301 Run, U101 TL072, U102 TL072, U201 L7805, U202 PT2399, U301 TL072

Commit message: -12Vc and Opamp removed on Clock sch
Parts:
- removed P301: HEADER_2x5_Doepfer, Connector_PinHeader_2.54mm:PinHeader_2x05_P2.54mm_Vertical
- added U302: LM555, AJ-Dropbox-Kicad:AJ_SO-8_5.3x6.2mm_P1.27mm, F.Cu at (247.0, 53.4)
- added U303: 4017, Package_SO:SOIC-16_4.55x10.3mm_P1.27mm, F.Cu at (237.8, 55.4)
- moved SW301 107.1 mm to (170.0, 113.2), turned to 90 degrees
- moved J313 99.1 mm to (189.0, 138.0), turned to 90 degrees
- moved J314 82.3 mm to (170.0, 101.5), turned to 270 degrees
- moved J301 82.1 mm to (170.0, 83.2), turned to 270 degrees
- moved J312 61.6 mm to (189.0, 128.9), turned to 90 degrees
- moved J304 58.1 mm to (189.0, 55.9), turned to 90 degrees
- moved J311 56.8 mm to (189.0, 119.8), turned to 90 degrees
- moved J307 54.6 mm to (189.0, 83.3), turned to 90 degrees
- moved J303 52.6 mm to (170.0, 92.4), turned to 270 degrees
- moved J308 49.5 mm to (189.0, 92.4), turned to 90 degrees
- moved RV301 48.6 mm to (162.5, 69.2)
- moved J309 47.4 mm to (189.0, 101.5), turned to 90 degrees
- moved J305 45.9 mm to (189.0, 65.0), turned to 90 degrees
- moved J310 45.2 mm to (189.0, 110.6), turned to 90 degrees
- moved J306 34.4 mm to (189.0, 74.2), turned to 90 degrees
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Connections:
- C309 pad 2: (no net) -> Net-(C309-Pad2)
- SW301 pad 2: (no net) -> Net-(SW301-Pad2)
