File: _saved_Kicad-EffectsUnit1.sch (KiCad schematic (older format))
At the start: 106 parts, among them J101 In7, J102 Doepfer connector, J104 In6, J105 In3, J106 Out10, J107 Out11, J108 Out9, J109 Out6, SW101 Dist 6, SW102 Crush A6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

Commit message: misc
Parts:
- D110, D111: footprint Diode_SMD:D_SOD-123 -> Diode_SMD:D_0805_2012Metric_Pad1.15x1.40mm_HandSolder
- D117: value LED_Out11 -> LED_11dist
- D118: value LED_CV2 -> LED_11dist; footprint LED_THT:LED_D3.0mm -> Diode_SMD:D_0805_2012Metric_Pad1.15x1.40mm_HandSolder
Changed lines of the file:
@@
 F 0 "D111" V 6375 2725 50  0000 L CNN
 F 1 "1N1007" V 6450 2725 50  0000 L CNN
-F 2 "Diode_SMD:D_SOD-123" H 6150 2925 50  0001 C CNN
+F 2 "Diode_SMD:D_0805_2012Metric_Pad1.15x1.40mm_HandSolder" H 6150 2925 50  0001 C CNN
 F 3 "~" H 6150 2925 50  0001 C CNN
 	1    6150 2925
@@
 F 0 "D110" V 5979 3004 50  0000 L CNN
 F 1 "1N1007" V 6070 3004 50  0000 L CNN
-F 2 "Diode_SMD:D_SOD-123" H 6025 2925 50  0001 C CNN
+F 2 "Diode_SMD:D_0805_2012Metric_Pad1.15x1.40mm_HandSolder" H 6025 2925 50  0001 C CNN
 F 3 "~" H 6025 2925 50  0001 C CNN
 	1    6025 2925
@@
 P 6150 4125
 F 0 "D118" H 6141 4341 50  0000 C CNN
-F 1 "LED_CV2" H 6141 4250 50  0000 C CNN
-F 2 "LED_THT:LED_D3.0mm" H 6150 4125 50  0001 C CNN
+F 1 "LED_11dist" H 6141 4250 50  0000 C CNN
+F 2 "Diode_SMD:D_0805_2012Metric_Pad1.15x1.40mm_HandSolder" H 6150 4125 50  0001 C CNN
 F 3 "~" H 6150 4125 50  0001 C CNN
 	1    6150 4125
@@
 P 6000 4125
 F 0 "D117" H 5991 4341 50  0000 C CNN
-F 1 "LED_Out11" H 5991 4250 50  0000 C CNN
+F 1 "LED_11dist" H 5991 4250 50  0000 C CNN
 F 2 "LED_SMD:LED_0805_2012Metric_Pad1.15x1.40mm_HandSolder" H 6000 4125 50  0001 C CNN
 F 3 "~" H 6000 4125 50  0001 C CNN
