File: Kicad-EffectsUnit1.sch (KiCad schematic (older format))
At the start: 104 parts, among them J101 In7, J102 Doepfer connector, J104 In6, J105 In3, J106 Out10, J107 Out11, J108 Out9, J109 Out6, SW101 Dist 6, SW102 Crush A6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

Commit message: filters
Parts:
- C117: value 33n -> 100n
- C122: value 44n -> 100n
- R111, R112, R117: value 11k -> 10k
- R115: value 110R -> 150R
- R119, R120: value 22k -> 10k
- R122: value 220R -> 150R
- R123: value 220R -> 10k
- R124: value 220k -> 10k
- R128: value 3k3 -> 10k
- R129, R132, R134: value 33k -> 10k
- R130: value 133R -> 150R
- R131: value 33k -> 220r
- R133: value 330k -> 10k
- R135, R136, R139: value 44k -> 10k
- R137: value 144R -> 150R
- R138: value 44k -> 220r
- R140: value 440k -> 10k
Changed lines of the file:
@@
 EESchema Schematic File Version 4
 LIBS:Kicad-EffectsUnit1-cache
-EELAYER 26 0
+EELAYER 29 0
 EELAYER END
 $Descr A4 11693 8268
@@
 P 4525 2225
 F 0 "R111" V 4318 2225 50  0000 C CNN
-F 1 "11k" V 4409 2225 50  0000 C CNN
+F 1 "10k" V 4409 2225 50  0000 C CNN
 F 2 "Resistor_SMD:R_0805_2012Metric_Pad1.15x1.40mm_HandSolder" V 4455 2225 50  0001 C CNN
 F 3 "~" H 4525 2225 50  0001 C CNN
@@
 P 4575 3400
 F 0 "R119" V 4368 3400 50  0000 C CNN
-F 1 "22k" V 4459 3400 50  0000 C CNN
+F 1 "10k" V 4459 3400 50  0000 C CNN
 F 2 "Resistor_SMD:R_0805_2012Metric_Pad1.15x1.40mm_HandSolder" V 4505 3400 50  0001 C CNN
 F 3 "~" H 4575 3400 50  0001 C CNN
@@
 P 5025 3400
 F 0 "R120" V 4818 3400 50  0000 C CNN
-F 1 "22k" V 4909 3400 50  0000 C CNN
+F 1 "10k" V 4909 3400 50  0000 C CNN
 F 2 "Resistor_SMD:R_0805_2012Metric_Pad1.15x1.40mm_HandSolder" V 4955 3400 50  0001 C CNN
 F 3 "~" H 5025 3400 50  0001 C CNN
@@
 P 4975 2225
 F 0 "R112" V 4768 2225 50  0000 C CNN
-F 1 "11k" V 4859 2225 50  0000 C CNN
+F 1 "10k" V 4650 2150 50  0000 C CNN
 F 2 "Resistor_SMD:R_0805_2012Metric_Pad1.15x1.40mm_HandSolder" V 4905 2225 50  0001 C CNN
 F 3 "~" H 4975 2225 50  0001 C CNN
@@
 P 4875 6575
 F 0 "R135" V 4668 6575 50  0000 C CNN
-F 1 "44k" V 4759 6575 50  0000 C CNN
+F 1 "10k" V 4759 6575 50  0000 C CNN
 F 2 "Resistor_SMD:R_0805_2012Metric_Pad1.15x1.40mm_HandSolder" V 4805 6575 50  0001 C CNN
 F 3 "~" H 4875 6575 50  0001 C CNN
@@
 P 5325 6575
 F 0 "R136" V 5118 6575 50  0000 C CNN
-F 1 "44k" V 5209 6575 50  0000 C CNN
+F 1 "10k" V 5209 6575 50  0000 C CNN
 F 2 "Resistor_SMD:R_0805_2012Metric_Pad1.15x1.40mm_HandSolder" V 5255 6575 50  0001 C CNN
 F 3 "~" H 5325 6575 50  0001 C CNN
@@
 P 4300 6975
 F 0 "R138" V 4093 6975 50  0000 C CNN
-F 1 "44k" V 4184 6975 50  0000 C CNN
+F 1 "220r" V 4184 6975 50  0000 C CNN
 F 2 "Resistor_SMD:R_0805_2012Metric_Pad1.15x1.40mm_HandSolder" V 4230 6975 50  0001 C CNN
 F 3 "~" H 4300 6975 50  0001 C CNN
@@
 P 4775 6975
 F 0 "R139" V 4568 6975 50  0000 C CNN
-F 1 "44k" V 4659 6975 50  0000 C CNN
+F 1 "10k" V 4659 6975 50  0000 C CNN
 F 2 "Resistor_SMD:R_0805_2012Metric_Pad1.15x1.40mm_HandSolder" V 4705 6975 50  0001 C CNN
 F 3 "~" H 4775 6975 50  0001 C CNN
@@
 U 1 1 5CCD4930
 P 5150 6300
-F 0 "C122" H 5050 6450 50  0000 L CNN
-F 1 "44n" H 5050 6550 50  0000 L CNN
+F 0 "C122" V 5050 6450 50  0000 L CNN
+F 1 "100n" V 4975 6550 50  0000 L CNN
 F 2 "Capacitor_SMD:C_0805_2012Metric_Pad1.15x1.40mm_HandSolder" H 5188 6150 50  0001 C CNN
 F 3 "~" H 5150 6300 50  0001 C CNN
@@
 P 4800 5050
 F 0 "R128" V 4593 5050 50  0000 C CNN
-F 1 "3k3" V 4684 5050 50  0000 C CNN
+F 1 "10k" V 4684 5050 50  0000 C CNN
 F 2 "Resistor_SMD:R_0805_2012Metric_Pad1.15x1.40mm_HandSolder" V 4730 5050 50  0001 C CNN
 F 3 "~" H 4800 5050 50  0001 C CNN
@@
 P 5825 5050
 F 0 "R129" V 5618 5050 50  0000 C CNN
-F 1 "33k" V 5709 5050 50  0000 C CNN
+F 1 "10k" V 5709 5050 50  0000 C CNN
 F 2 "Resistor_SMD:R_0805_2012Metric_Pad1.15x1.40mm_HandSolder" V 5755 5050 50  0001 C CNN
 F 3 "~" H 5825 5050 50  0001 C CNN
@@
 P 4300 5450
 F 0 "R131" V 4093 5450 50  0000 C CNN
-F 1 "33k" V 4184 5450 50  0000 C CNN
+F 1 "220r" V 4184 5450 50  0000 C CNN
 F 2 "Resistor_SMD:R_0805_2012Metric_Pad1.15x1.40mm_HandSolder" V 4230 5450 50  0001 C CNN
 F 3 "~" H 4300 5450 50  0001 C CNN
@@
 P 4775 5450
 F 0 "R132" V 4568 5450 50  0000 C CNN
-F 1 "33k" V 4659 5450 50  0000 C CNN
+F 1 "10k" V 4659 5450 50  0000 C CNN
 F 2 "Resistor_SMD:R_0805_2012Metric_Pad1.15x1.40mm_HandSolder" V 4705 5450 50  0001 C CNN
 F 3 "~" H 4775 5450 50  0001 C CNN
@@
 U 1 1 5CE1CD69
 P 5150 4775
-F 0 "C117" H 5050 4925 50  0000 L CNN
-F 1 "33n" H 5050 5025 50  0000 L CNN
+F 0 "C117" V 5225 4900 50  0000 L CNN
+F 1 "100n" V 5100 4950 50  0000 L CNN
 F 2 "Capacitor_SMD:C_0805_2012Metric_Pad1.15x1.40mm_HandSolder" H 5188 4625 50  0001 C CNN
 F 3 "~" H 5150 4775 50  0001 C CNN
@@
 P 5725 2775
 F 0 "R115" V 5518 2775 50  0000 C CNN
-F 1 "110R" V 5609 2775 50  0000 C CNN
+F 1 "150R" V 5609 2775 50  0000 C CNN
 F 2 "Resistor_SMD:R_0805_2012Metric_Pad1.15x1.40mm_HandSolder" V 5655 2775 50  0001 C CNN
 F 3 "~" H 5725 2775 50  0001 C CNN
@@
 P 5775 3950
 F 0 "R122" V 5568 3950 50  0000 C CNN
-F 1 "220R" V 5659 3950 50  0000 C CNN
+F 1 "150R" V 5659 3950 50  0000 C CNN
 F 2 "Resistor_SMD:R_0805_2012Metric_Pad1.15x1.40mm_HandSolder" V 5705 3950 50  0001 C CNN
 F 3 "~" H 5775 3950 50  0001 C CNN
@@
 P 6050 5350
 F 0 "R130" V 5843 5350 50  0000 C CNN
-F 1 "133R" V 5934 5350 50  0000 C CNN
+F 1 "150R" V 5934 5350 50  0000 C CNN
 F 2 "Resistor_SMD:R_0805_2012Metric_Pad1.15x1.40mm_HandSolder" V 5980 5350 50  0001 C CNN
 F 3 "~" H 6050 5350 50  0001 C CNN
@@
 P 6050 6875
 F 0 "R137" V 5843 6875 50  0000 C CNN
-F 1 "144R" V 5934 6875 50  0000 C CNN
+F 1 "150R" V 5934 6875 50  0000 C CNN
 F 2 "Resistor_SMD:R_0805_2012Metric_Pad1.15x1.40mm_HandSolder" V 5980 6875 50  0001 C CNN
 F 3 "~" H 6050 6875 50  0001 C CNN
@@
 U 1 1 5CCC0D3E
 P 4975 2350
-F 0 "D106" V 4929 2429 50  0000 L CNN
-F 1 "1N1007" V 5020 2429 50  0000 L CNN
+F 0 "D106" V 4825 2250 50  0000 L CNN
+F 1 "1N1007" V 4700 2150 50  0000 L CNN
 F 2 "Diode_SMD:D_SOD-123" H 4975 2350 50  0001 C CNN
 F 3 "~" H 4975 2350 50  0001 C CNN
@@
 U 1 1 5CCC0ECC
 P 4975 2475
-F 0 "D108" V 4929 2554 50  0000 L CNN
-F 1 "1N1007" V 5020 2554 50  0000 L CNN
+F 0 "D108" V 5150 2525 50  0000 L CNN
+F 1 "1N1007" V 5250 2575 50  0000 L CNN
 F 2 "Diode_SMD:D_SOD-123" H 4975 2475 50  0001 C CNN
 F 3 "~" H 4975 2475 50  0001 C CNN
@@
 P 6700 2975
 F 0 "R117" V 6493 2975 50  0000 C CNN
-F 1 "11k" V 6584 2975 50  0000 C CNN
+F 1 "10k" V 6584 2975 50  0000 C CNN
 F 2 "Resistor_SMD:R_0805_2012Metric_Pad1.15x1.40mm_HandSolder" V 6630 2975 50  0001 C CNN
 F 3 "~" H 6700 2975 50  0001 C CNN
@@
 P 4300 5600
 F 0 "R133" V 4475 5575 50  0000 C CNN
-F 1 "330k" V 4400 5600 50  0000 C CNN
+F 1 "10k" V 4400 5600 50  0000 C CNN
 F 2 "Resistor_SMD:R_0805_2012Metric_Pad1.15x1.40mm_HandSolder" V 4230 5600 50  0001 C CNN
 F 3 "~" H 4300 5600 50  0001 C CNN
@@
 P 4675 4175
 F 0 "R124" V 4850 4150 50  0000 C CNN
-F 1 "220k" V 4775 4175 50  0000 C CNN
+F 1 "10k" V 4775 4175 50  0000 C CNN
 F 2 "Resistor_SMD:R_0805_2012Metric_Pad1.15x1.40mm_HandSolder" V 4605 4175 50  0001 C CNN
 F 3 "~" H 4675 4175 50  0001 C CNN
@@
 P 4675 4050
 F 0 "R123" V 4468 4050 50  0000 C CNN
-F 1 "220R" V 4559 4050 50  0000 C CNN
+F 1 "10k" V 4559 4050 50  0000 C CNN
 F 2 "Resistor_SMD:R_0805_2012Metric_Pad1.15x1.40mm_HandSolder" V 4605 4050 50  0001 C CNN
 F 3 "~" H 4675 4050 50  0001 C CNN
@@
 P 4300 7150
 F 0 "R140" V 4475 7150 50  0000 C CNN
-F 1 "440k" V 4400 7150 50  0000 C CNN
+F 1 "10k" V 4400 7150 50  0000 C CNN
 F 2 "Resistor_SMD:R_0805_2012Metric_Pad1.15x1.40mm_HandSolder" V 4230 7150 50  0001 C CNN
 F 3 "~" H 4300 7150 50  0001 C CNN
@@
 P 6325 5950
 F 0 "R134" H 6200 6025 50  0000 C CNN
-F 1 "33k" H 6209 5950 50  0000 C CNN
+F 1 "10k" H 6209 5950 50  0000 C CNN
 F 2 "Resistor_SMD:R_0805_2012Metric_Pad1.15x1.40mm_HandSolder" V 6255 5950 50  0001 C CNN
 F 3 "~" H 6325 5950 50  0001 C CNN

Commit message: filters 2
Parts:
- C123: value 44n -> 33n
Changed lines of the file:
@@
 P 5050 7175
 F 0 "C123" H 4950 7325 50  0000 L CNN
-F 1 "44n" H 4950 7425 50  0000 L CNN
+F 1 "33n" H 4950 7425 50  0000 L CNN
 F 2 "Capacitor_SMD:C_0805_2012Metric_Pad1.15x1.40mm_HandSolder" H 5088 7025 50  0001 C CNN
 F 3 "~" H 5050 7175 50  0001 C CNN
