File: Kicad-EffectsUnit1.sch (KiCad schematic (older format))
At the start: 104 parts, among them J101 In7, J102 Doepfer connector, J104 In6, J105 In3, J106 Out10, J107 Out11, J108 Out9, J109 Out6, SW101 Dist 6, SW102 Crush A6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

Commit message: Rev B initiated
Parts:
- added R?: 10k, Resistor_SMD:R_0805_2012Metric_Pad1.15x1.40mm_HandSolder, symbol Device:R
- RV104: value 10k_A4 -> 100k_A4
- RV105: value 10k_A5 -> 100k_A5
Connections:
- net GND: now also R?.2; no longer D117.1 (K), D118.2 (A)
- net Out10Dist: now also R134.2
- net at SW105.4 (A): no longer R134.2
- new net: D117.1 (K), D118.2 (A), R?.1
Other:
- moved on the sheet: R134
Changed lines of the file:
@@
 Sheet 1 3
 Title "Effects Unit 1"
-Date "2019-02-05"
-Rev "Rev 1"
+Date "2019-04-25"
+Rev "Rev B"
 Comp "Promesoft"
 Comment1 "Johansen Engineering"
@@
 L power:GND #PWR0110
 U 1 1 5D28C9A9
-P 6150 4350
-F 0 "#PWR0110" H 6150 4100 50  0001 C CNN
-F 1 "GND" H 6155 4177 50  0000 C CNN
-F 2 "" H 6150 4350 50  0001 C CNN
-F 3 "" H 6150 4350 50  0001 C CNN
-	1    6150 4350
+P 6500 4350
+F 0 "#PWR0110" H 6500 4100 50  0001 C CNN
+F 1 "GND" H 6505 4177 50  0000 C CNN
+F 2 "" H 6500 4350 50  0001 C CNN
+F 3 "" H 6500 4350 50  0001 C CNN
+	1    6500 4350
 	1    0    0    -1
 $EndComp
@@
 Text GLabel 6250 3950 2    50   Input ~ 0
 Out11Dist
-Text GLabel 6350 5350 2    50   Input ~ 0
+Text GLabel 6625 5350 2    50   Input ~ 0
 Out10Dist
-Wire Wire Line
-	6150 4275 6150 4350
 Wire Wire Line
 	2125 5600 2125 5575
@@
 U 2 1 5D49153E
 P 6225 5550
-F 0 "SW105" V 6179 5698 50  0000 L CNN
-F 1 "Dist 10" V 6270 5698 50  0000 L CNN
+F 0 "SW105" V 6175 5325 50  0000 L CNN
+F 1 "Dist 10" V 6250 5325 50  0000 L CNN
 F 2 "AJ-Dropbox-Kicad:SPDTx2" H 6225 5550 50  0001 C CNN
 F 3 "~" H 6225 5550 50  0001 C CNN
@@
 L Device:R R134
 U 1 1 5D4EE5BD
-P 6325 5950
-F 0 "R134" H 6150 6025 50  0000 C CNN
-F 1 "10k" H 6150 5950 50  0000 C CNN
-F 2 "Resistor_SMD:R_0805_2012Metric_Pad1.15x1.40mm_HandSolder" V 6255 5950 50  0001 C CNN
-F 3 "~" H 6325 5950 50  0001 C CNN
-	1    6325 5950
+P 6500 5600
+F 0 "R134" H 6325 5675 50  0000 C CNN
+F 1 "10k" H 6400 5800 50  0000 C CNN
+F 2 "Resistor_SMD:R_0805_2012Metric_Pad1.15x1.40mm_HandSolder" V 6430 5600 50  0001 C CNN
+F 3 "~" H 6500 5600 50  0001 C CNN
+	1    6500 5600
 	-1   0    0    1
 $EndComp
-Wire Wire Line
-	6325 5750 6325 5800
-Wire Wire Line
-	6175 5800 6250 5800
-Wire Wire Line
-	6250 5800 6250 6100
-Wire Wire Line
-	6250 6100 6325 6100
 Connection ~ 6175 5800
 $Comp
@@
 Wire Wire Line
 	6100 6100 6175 6100
-Wire Wire Line
-	6225 5350 6350 5350
 Wire Wire Line
 	1850 5350 1850 5375
@@
 P 7900 5075
 F 0 "RV104" V 7525 5225 50  0000 R CNN
-F 1 "10k_A4" V 7625 5250 50  0000 R CNN
+F 1 "100k_A4" V 7625 5250 50  0000 R CNN
 F 2 "Potentiometer_THT:Potentiometer_China_RK09_Single_Vertical_AJ" H 7900 5075 50  0001 C CNN
 F 3 "~" H 7900 5075 50  0001 C CNN
@@
 P 7900 5625
 F 0 "RV105" V 7750 5800 50  0000 R CNN
-F 1 "10k_A5" V 7675 5700 50  0000 R CNN
+F 1 "100k_A5" V 7675 5700 50  0000 R CNN
 F 2 "Potentiometer_THT:Potentiometer_China_RK09_Single_Vertical_AJ" H 7900 5625 50  0001 C CNN
 F 3 "~" H 7900 5625 50  0001 C CNN
@@
 F1 "EU3.sch" 50
 $EndSheet
+Wire Wire Line
+	6500 5800 6500 5750
+Wire Wire Line
+	6500 5450 6500 5350
+Wire Wire Line
+	6175 5800 6500 5800
+Wire Wire Line
+	6225 5350 6500 5350
+Wire Wire Line
+	6625 5350 6500 5350
+Connection ~ 6500 5350
+$Comp
+L Device:R R?
+U 1 1 5CCAB2D3
+P 6300 4275
+F 0 "R?" H 6125 4350 50  0000 C CNN
+F 1 "10k" H 6200 4475 50  0000 C CNN
+F 2 "Resistor_SMD:R_0805_2012Metric_Pad1.15x1.40mm_HandSolder" V 6230 4275 50  0001 C CNN
+F 3 "~" H 6300 4275 50  0001 C CNN
+	1    6300 4275
+	0    -1   -1   0
+$EndComp
+Wire Wire Line
+	6450 4275 6500 4275
+Wire Wire Line
+	6500 4275 6500 4350
 $EndSCHEMATC

Commit message: Switch 1/2 rev
Parts:
- RV101: value 10k_O6 -> 20k_O6
- RV102: value 10k_O11 -> 20k_O11
Connections:
- net at R115.2, RV101.2, RV101.3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: now also SW101.3 (C); no longer SW101.1 (A)
Changed lines of the file:
@@
 P 5375 3400
 F 0 "RV102" H 5305 3446 50  0000 R CNN
-F 1 "10k_O11" H 5305 3355 50  0000 R CNN
+F 1 "20k_O11" H 5305 3355 50  0000 R CNN
 F 2 "Potentiometer_THT:Potentiometer_China_RK09_Single_Vertical_AJ" H 5375 3400 50  0001 C CNN
 F 3 "~" H 5375 3400 50  0001 C CNN
@@
 P 5325 2225
 F 0 "RV101" V 5525 2300 50  0000 R CNN
-F 1 "10k_O6" V 5425 2200 50  0000 R CNN
+F 1 "20k_O6" V 5425 2200 50  0000 R CNN
 F 2 "Potentiometer_THT:Potentiometer_China_RK09_Single_Vertical_AJ" H 5325 2225 50  0001 C CNN
 F 3 "~" H 5325 2225 50  0001 C CNN
@@
 	5475 2225 5575 2225
 Wire Wire Line
-	5575 2225 5575 2300
-Wire Wire Line
 	5625 3400 5625 3950
 Connection ~ 5625 3950
@@
 Wire Wire Line
 	5125 2400 5125 2350
-Wire Wire Line
-	5525 2300 5575 2300
-Connection ~ 5575 2300
-Wire Wire Line
-	5575 2300 5575 2775
 $Comp
 L Device:LED D118
@@
 Wire Wire Line
 	6500 4275 6500 4350
+Wire Wire Line
+	5525 2500 5575 2500
+Connection ~ 5575 2500
+Wire Wire Line
+	5575 2500 5575 2775
+Wire Wire Line
+	5575 2225 5575 2500
 $EndSCHEMATC
